File: hardware/touch-kit/music-kit.kicad_sch (KiCad schematic)
At the start: 0 parts

Commit message: pcb finished
Parts:
- added BT1, BT2: Push_Button_W12mm, PCM_SL_Footprints:Push_Button_W12mm, symbol PCM_SL_Devices:Push_Button_W12mm
- added ENC1: RotaryEncoder_Switch_MP, Rotary_Encoder:RotaryEncoder_Alps_EC11E-Switch_Vertical_H20mm, symbol Device:RotaryEncoder_Switch_MP
- added H1, H2, H3, H4: MountingHole_Pad, MountingHole:MountingHole_3.2mm_M3_DIN965_Pad, symbol Mechanical:MountingHole_Pad
- added J1: Power, Connector_PinSocket_2.54mm:PinSocket_1x02_P2.54mm_Horizontal, symbol Connector:Conn_01x02_Pin
- added J12, J3: DAC_JUMPPER, Connector_PinHeader_2.54mm:PinHeader_1x02_P2.54mm_Vertical, symbol Connector:Conn_01x02_Pin
- added J4: Speakerdf, Connector_PinSocket_2.54mm:PinSocket_1x03_P2.54mm_Vertical, symbol Connector:Conn_01x03_Socket
- added J5: INPUTS, Connector_JST:JST_XH_B8B-XH-A_1x08_P2.50mm_Vertical, symbol Connector:Conn_01x08_Pin
- added J6: Power Conn, Connector_JST:JST_XH_B2B-XH-A_1x02_P2.50mm_Vertical, symbol Connector:Conn_01x02_Pin
- added JP1, JP2, JP3: SolderJumper_3_Bridged12, Jumper:SolderJumper-3_P1.3mm_Bridged12_Pad1.0x1.5mm, symbol Jumper:SolderJumper_3_Bridged12
- added JP4: SolderJumper_2_Bridged, Jumper:SolderJumper-2_P1.3mm_Bridged_Pad1.0x1.5mm, symbol Jumper:SolderJumper_2_Bridged
- added LED1: NEOPIXEL, Connector_PinSocket_2.54mm:PinSocket_1x03_P2.54mm_Vertical, symbol Connector:Conn_01x03_Socket
- added PAM1: PAM8403, Connector_PinHeader_2.54mm:PinHeader_1x11_P2.54mm_Vertical, symbol Connector:Conn_01x11_Pin
- added SW1: Slide_Switch_SPDT_P3mm_10x5x10mm, PCM_SL_Devices:Slide_Switch_SPDT_P3mm_10x5x10mm, symbol PCM_SL_Devices:Slide_Switch_SPDT_P3mm_10x5x10mm
- added U1: LM1117T-3.3, Package_TO_SOT_THT:TO-220-3_Horizontal_TabDown, symbol Regulator_Linear:LM1117T-3.3
- added U2: ESP32-DevKitC, PCM_Espressif:ESP32-DevKitC, symbol PCM_Espressif:ESP32-DevKitC
- added U3: ER_OLEDM0.91_1x-I2C, Display:ER_OLEDM0.91_1x-I2C, symbol Display_Graphic:ER_OLEDM0.91_1x-I2C
Connections:
- new net: JP3.2 (C), LED1.1 (Pin_1)
- new net: JP2.2 (C), U3.1 (GND)
- new net: JP1.2 (C), U3.2 (VCC)
- new net: SW1.2, U1.3 (VI)
- new net: JP4.2 (B), U2.19 (5V)
- new net +BATT: J1.2 (Pin_2), JP3.3 (B), JP4.1 (A), SW1.1
- new net AUDIO_OUT+: J12.2 (Pin_2), PAM1.3 (Pin_3)
- new net AUDIO_OUT-: J12.1 (Pin_1), PAM1.4 (Pin_4)
- new net BT1: BT1.1, U2.27 (GPIO16)
- new net BT2: BT2.1, U2.28 (GPIO17)
- new net DAC_MCU: J3.1 (Pin_1), U2.9 (DAC_1/ADC2_CH8/GPIO25)
- new net DAC_OUT: J3.2 (Pin_2), J4.1 (Pin_1), PAM1.9 (Pin_9)
- new net ENC_CLK: ENC1.A, U2.31 (GPIO19)
- new net ENC_DT: ENC1.B, U2.30 (GPIO18)
- new net ENC_SW: ENC1.S1, U2.29 (GPIO5)
- new net GND: BT1.2, BT2.2, ENC1.C, ENC1.S2, H1.1, H2.1, H3.1, H4.1, J1.1 (Pin_1), J4.3 (Pin_3), J5.8 (Pin_8), J6.2 (Pin_2), JP1.3 (B), JP2.1 (A), LED1.3 (Pin_3), PAM1.10 (Pin_10), PAM1.6 (Pin_6), U1.1 (GND), U2.14 (GND), U2.32 (GND), U2.38 (GND)
- new net S1: J5.1 (Pin_1), U2.26 (ADC2_CH0/GPIO4)
- new net S2: J5.2 (Pin_2), U2.23 (MTDO/GPIO15/ADC2_CH3)
- new net S3: J5.3 (Pin_3), U2.15 (MTCK/GPIO13/ADC2_CH4)
- new net S4: J5.4 (Pin_4), U2.12 (MTMS/GPIO14/ADC2_CH6)
- new net S5: J5.5 (Pin_5), U2.11 (ADC2_CH7/GPIO27)
- new net S6: J5.6 (Pin_6), U2.8 (32K_XN/GPIO33/ADC1_CH5)
- new net S7: J5.7 (Pin_7), U2.7 (32K_XP/GPIO32/ADC1_CH4)
- new net SCL: U2.36 (GPIO22), U3.3 (SCL)
- new net SDA: U2.33 (GPIO21), U3.4 (SDA)
- new net VCC: J4.2 (Pin_2), J6.1 (Pin_1), JP1.1 (A), JP2.3 (B), JP3.1 (A), PAM1.7 (Pin_7), U1.2 (VO), U2.1 (3V3)
- new net WS_DATA: LED1.2 (Pin_2), U2.10 (DAC_2/ADC2_CH9/GPIO26)
Other:
- note added: "CONTROLS"
- note added: "MOUNTING HOLES"
- note added: "POWER"
